File: EPS.kicad_sch (KiCad schematic)
At the start: 91 parts, among them IC1 TPS22997RYZR, IC10 SN65HVD1782QDRQ1, IC11 MCP2518FDT-E_SL, IC12 MCP2518FDT-E_SL, IC2 TPS56C230RJER, IC3 TPS22997RYZR, IC7 TPS22997RYZR, IC8 TPS22997RYZR, IC9 TCAN1046AVDYYRQ1, J1 S4B-XH-A_LF__SN_, J2 PH1RA-02-UA, J4 M80-5000000M1-04-333-00-000, Q1 SI4497DY-T1-GE3, U1 INA260, U2 INA260, U3 INA260, U4 INA260, U5 INA260, Y1 40MHz, Y2 40MHz

Commit message: updated schematic, began revising routing
Parts:
- removed C28: 100n, Capacitor_SMD:C_0603_1608Metric, symbol Device:C_Small
- removed D9: SM712-02HTG, HEDGE2-EPS:SM71202HTG, symbol HEDGE2:SM712-02HTG
- removed IC10: SN65HVD1782QDRQ1, HEDGE2-EPS:SN65HVD1782QDRQ1, symbol HEDGE2:SN65HVD1782QDRQ1
- removed J2: PH1RA-02-UA, HEDGE2-EPS:PH1RA02UA, symbol HEDGE2:PH1RA-02-UA
- removed R18, R19: 60, Resistor_SMD:R_0603_1608Metric, symbol Device:R_Small_US
- removed R20, R21: 10k, Resistor_SMD:R_0603_1608Metric, symbol Device:R_Small_US
- removed R22, R23: 10, Resistor_SMD:R_0603_1608Metric, symbol Device:R_Small_US
- added IC4: TPS22997RYZR, HEDGE2-EPS:TPS22997RYZR, symbol HEDGE2:TPS22997RYZR
- added R13, R14, R15: 10k, Resistor_SMD:R_0603_1608Metric, symbol Device:R_Small_US
- added S1: SS-5D, HEDGE2-EPS:SS5D, symbol HEDGE2:SS-5D
- added U6: INA260, Package_SO:TSSOP-16_4.4x5mm_P0.65mm, symbol Sensor:INA260
- C24: value 100n -> 1n
- R11: value 4k7 -> 1k
- R12: value 2k2 -> 330
- R16, R17: value 60 -> 10k
Connections:
- net +3V3: now also C26.1, U6.10 (VS), U6.4 (A1), U6.5 (A0); no longer C24.1, C9.1
- net +5V: now also R12.1, U6.1 (IN+), U6.12 (VBUS), U6.2 (IN+), U6.3 (IN+); no longer D3.2 (A)
- net +BATT_SENSE: now also R11.1; no longer D4.2 (A)
- net CAN_A_H: no longer R16.1
- net CAN_A_L: no longer R17.2
- net GND: now also D3.1 (K), D4.1 (K), IC4.5 (GND), U6.11 (GND), U6.6 (GND); no longer R11.2, R12.2
- net GNSS_C: now also R14.2; no longer A1.17 (GPIO13), IC8.10 (ON)
- net OBC_C: now also R13.2; no longer A1.16 (GPIO12), IC1.10 (ON)
- net SCI_C: now also R15.2; no longer A1.19 (GPIO14), IC3.10 (ON)
- net SCL: now also U6.9 (SCL)
- net SDA: now also U6.8 (SDA)
- net +5V_COMM_DMR: now reaches H1EPS1.51
- net +5V_COMM_DMR: now also IC4.6 (QOD), IC4.7 (VOUT_1), IC4.8 (VOUT_2)
- net +5V_COMM renamed +5V_COMM_XBEE
- net +5V_COMM_SENSE renamed +5V_COMM_XBEE_SENSE
- net AD0/DIO0_XB: no longer names the net of H2EPS1.15
- net AD1/DIO1/SPI_ATTN_XB: no longer names the net of H2EPS1.10
- net AD3/DIO3/SPI_SSEL_XB: no longer names the net of H2EPS1.05
- net AD/DIO2/SPI_CLK_XB: no longer names the net of H2EPS1.06
- net COMM_C: no longer names the net of A1.20 (GPIO15)
- net COMM_C: no longer IC7.10 (ON)
- net CS_DMR: no longer names the net of H2EPS1.24
- net CTS/DIO7_XB: no longer names the net of H2EPS1.04
- net DIO10/PWM0_XB: no longer names the net of H2EPS1.12
- net DIO11/PWM1_XB: no longer names the net of H2EPS1.14
- net DIO12/SPI_MISO_XB: no longer names the net of H2EPS1.08
- net DIO4/SPI_MOSI_XB: no longer names the net of H2EPS1.07
- net EN: no longer names the net of D1.1 (K), IC2.12 (EN), R6.2, R7.1
- net HST_RXD_DMR: no longer names the net of H2EPS1.25
- net HST_TXD_DMR: no longer names the net of H2EPS1.27
- net NDTR_XB: no longer names the net of H2EPS1.17
- net RS485_E: no longer names the net of A1.10 (GPIO7)
- net RS485_RX: no longer names the net of A1.12 (GPIO9)
- net RS485_TX: no longer names the net of A1.11 (GPIO8)
- net RTS/DIO6_XB: no longer names the net of H2EPS1.03
- net SPKEN_DMR: no longer names the net of H2EPS1.23
- net UART_G_RX (EPS): no longer names the net of H1EPS1.43
- net UART_G_TX (EPS): no longer names the net of H1EPS1.41
- new net: IC1.10 (ON), R13.1
- new net: D4.2 (A), R11.2
- new net: IC8.10 (ON), R14.1
- new net: IC4.10 (ON), R17.1
- new net: D3.2 (A), R12.2
- new net: IC7.10 (ON), R16.1
- new net: C24.1, IC4.9 (CT)
- new net: IC3.10 (ON), R15.1
- new net +5V_COMM_DMR_SENSE: C9.1, IC4.1 (VBIAS), IC4.2 (VIN_1), IC4.3 (VIN_2), U6.14 (IN-), U6.15 (IN-), U6.16 (IN-)
- new net COMM_DMR_C: R17.2
- new net COMM_XBEE_C: R16.2
- no-connect marks 85 -> 106
Other:
- note added: "2V Voltage Drop, 10 mA"
- note removed: "Battery/Step Down Converter Inhibit"
- note removed: "RS485 Communication"
- moved on the sheet: C12, C13, C14, C15, C16, C17, C18, C19, C20, C21, C22, C23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

Commit message: implemented updates
Parts:
- D3, D4: footprint LED_SMD:LED_0603_1608Metric -> LED_THT:LED_D3.0mm
- R11: value 1k -> 820; footprint Resistor_SMD:R_0603_1608Metric -> Resistor_SMD:R_0805_2012Metric
- R12: footprint Resistor_SMD:R_0603_1608Metric -> Resistor_SMD:R_0805_2012Metric
Connections:
- net +5V_COMM_DMR: now also IC7.6 (QOD), IC7.7 (VOUT_1), IC7.8 (VOUT_2); no longer IC4.6 (QOD), IC4.7 (VOUT_1), IC4.8 (VOUT_2)
- net +5V_COMM_DMR_SENSE: now also C19.1, IC7.1 (VBIAS), IC7.2 (VIN_1), IC7.3 (VIN_2), U5.14 (IN-), U5.15 (IN-), U5.16 (IN-); no longer C9.1, IC4.1 (VBIAS), IC4.2 (VIN_1), IC4.3 (VIN_2), U6.14 (IN-), U6.15 (IN-), U6.16 (IN-)
- net +5V_COMM_XBEE: now also IC3.6 (QOD), IC3.7 (VOUT_1), IC3.8 (VOUT_2); no longer IC7.6 (QOD), IC7.7 (VOUT_1), IC7.8 (VOUT_2)
- net +5V_COMM_XBEE_SENSE: now also C17.1, IC3.1 (VBIAS), IC3.2 (VIN_1), IC3.3 (VIN_2), U2.14 (IN-), U2.15 (IN-), U2.16 (IN-); no longer C19.1, IC7.1 (VBIAS), IC7.2 (VIN_1), IC7.3 (VIN_2), U5.14 (IN-), U5.15 (IN-), U5.16 (IN-)
- net +5V_GNSS: now also IC1.6 (QOD), IC1.7 (VOUT_1), IC1.8 (VOUT_2); no longer IC8.6 (QOD), IC8.7 (VOUT_1), IC8.8 (VOUT_2)
- net +5V_GNSS_SENSE: now also C15.1, IC1.1 (VBIAS), IC1.2 (VIN_1), IC1.3 (VIN_2), U1.14 (IN-), U1.15 (IN-), U1.16 (IN-); no longer C21.1, IC8.1 (VBIAS), IC8.2 (VIN_1), IC8.3 (VIN_2), U4.14 (IN-), U4.15 (IN-), U4.16 (IN-)
- net +5V_OBC: now also IC4.6 (QOD), IC4.7 (VOUT_1), IC4.8 (VOUT_2); no longer IC1.6 (QOD), IC1.7 (VOUT_1), IC1.8 (VOUT_2)
- net +5V_OBC_SENSE: now also C9.1, IC4.1 (VBIAS), IC4.2 (VIN_1), IC4.3 (VIN_2), U6.14 (IN-), U6.15 (IN-), U6.16 (IN-); no longer C15.1, IC1.1 (VBIAS), IC1.2 (VIN_1), IC1.3 (VIN_2), U1.14 (IN-), U1.15 (IN-), U1.16 (IN-)
- net +5V_SCI: now also IC8.6 (QOD), IC8.7 (VOUT_1), IC8.8 (VOUT_2); no longer IC3.6 (QOD), IC3.7 (VOUT_1), IC3.8 (VOUT_2)
- net +5V_SCI_SENSE: now also C21.1, IC8.1 (VBIAS), IC8.2 (VIN_1), IC8.3 (VIN_2), U4.14 (IN-), U4.15 (IN-), U4.16 (IN-); no longer C17.1, IC3.1 (VBIAS), IC3.2 (VIN_1), IC3.3 (VIN_2), U2.14 (IN-), U2.15 (IN-), U2.16 (IN-)
- net COMM_DMR_C: now also A1.20 (GPIO15), R16.2; no longer R17.2
- net COMM_XBEE_C: now also A1.19 (GPIO14), R15.2; no longer R16.2
- net GNSS_C: now also A1.16 (GPIO12), R13.2; no longer R14.2
- net OBC_C: now also A1.15 (GPIO11), R17.2; no longer R13.2
- net SCI_C: now also A1.17 (GPIO13), R14.2; no longer R15.2
- net +BATT_BIN: now reaches S1.1 (COM)
- net +BATT_BIN: now also BT3.P, J1.4
- net +BATT_AIN: now reaches S1.3 (NC)
- net +BATT_AIN: now also J4.A2, J4.A4
- removed net +BATT_BSW: BT3.P, J1.4, J4.A2, J4.A4
Other:
- note added: "2V Voltage Drop, ~10 mA"
- note removed: "2V Voltage Drop, 10 mA"
- moved on the sheet: BT1, BT2, BT3, C18, C19, C20, C21, C22, C24, C9, IC4, IC7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
