File: EPS.kicad_sch (KiCad schematic)
At the start: 87 parts, among them IC1 TPS22997RYZR, IC11 MCP2518FDT-E_SL, IC12 MCP2518FDT-E_SL, IC2 TPS56C230RJER, IC3 TPS22997RYZR, IC4 TPS22997RYZR, IC7 TPS22997RYZR, IC8 TPS22997RYZR, IC9 TCAN1046AVDYYRQ1, J1 S4B-XH-A_LF__SN_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

Commit message: updated bom
Parts:
- A1: value RaspberryPi_Pico -> RaspberryPi_Pico 2; DigiKey Part Number (none) -> 2648-SC1631CT-ND
- BT1, BT2, BT3: DigiKey Part Number (none) -> 36-1043-ND
- D1: value Zener -> Zener 5v1; DigiKey Part Number (none) -> MMSZ5231B-FDICT-ND
- D2: value Schottky -> Schottky 1A; DigiKey Part Number (none) -> MBR130LSFT1GOSCT-ND
- D3, D4: DigiKey Part Number (none) -> 732-5005-ND
- IC1, IC3, IC4, IC7, IC8: DigiKey Part Number (none) -> 296-TPS22997RYZRCT-ND
- IC11, IC12: DigiKey Part Number (none) -> MCP2518FDT-E/SLCT-ND
- IC2: DigiKey Part Number (none) -> 296-TPS56C230RJERCT-ND
- IC9: DigiKey Part Number (none) -> 296-TCAN1046AVDYYRQ1CT-ND
- J1: DigiKey Part Number (none) -> 455-2243-ND
- J4: DigiKey Part Number (none) -> Mouser 855-0000M10433300000
- L1: DigiKey Part Number (none) -> 732-744393465033CT-ND
- MH1, MH2, MH3, MH4: DigiKey Part Number (none) -> NA
- Q1: DigiKey Part Number (none) -> SI4497DY-T1-GE3CT-ND
- S1: DigiKey Part Number (none) -> SW241-ND
- U1, U2, U3, U4, U5, U6: DigiKey Part Number (none) -> 296-47777-1-ND
- Y1, Y2: DigiKey Part Number (none) -> 535-15281-1-ND
Other:
- moved on the sheet: C1, C2, C3, C4, C5, C6, IC2, L1, R1, R2, R3, R4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
